Commit message: Initial Commit

File: ur5_description/urdf/ur5.urdf.xacro (robot description, xacro)
@@ -76,4 +76,5 @@
           <color rgba="0.7 0.7 0.7 1.0"/>
         </material>
+        <origin xyz="-0.02 0.86 0.7" rpy="-2.72 -0.11 0.57" />
       </visual>
       <collision>
@@ -83,5 +84,5 @@
       </collision>
       <xacro:cylinder_inertial radius="0.06" length="0.05" mass="${base_mass}">
-        <origin xyz="0.0 0.0 0.0" rpy="0 0 0" />
+        <origin xyz="0.0 0.0 1.0" rpy="0 0 0" />
       </xacro:cylinder_inertial>
     </link>
@@ -89,5 +90,5 @@
       <parent link="${prefix}base_link" />
       <child link = "${prefix}shoulder_link" />
-      <origin xyz="0.0 0.0 ${shoulder_height}" rpy="0.0 0.0 0.0" />
+      <origin xyz="-0.02 0.86 0.7" rpy="-2.72 -0.11 0.57" />
       <axis xyz="0 0 1" />
       <xacro:unless value="${joint_limited}">
@@ -288,14 +289,14 @@
     <xacro:ur_arm_gazebo prefix="${prefix}" />
     <!-- ROS base_link to UR 'Base' Coordinates transform -->
-    <link name="${prefix}base"/>
-    <joint name="${prefix}base_link-base_fixed_joint" type="fixed">
+    <!-- <link name="${prefix}base"/> -->
+    <!-- <joint name="${prefix}base_link-base_fixed_joint" type="fixed"> -->
       <!-- NOTE: this rotation is only needed as long as base_link itself is
                  not corrected wrt the real robot (ie: rotated over 180
                  degrees)
       -->
-      <origin xyz="0 0 0" rpy="0 0 ${-pi}"/>
-      <parent link="${prefix}base_link"/>
-      <child link="${prefix}base"/>
-    </joint>
+      <!-- <origin xyz="0 0 2.0" rpy="0.0 0 ${-pi}"/> -->
+      <!-- <parent link="${prefix}base_link"/> -->
+      <!-- <child link="${prefix}base"/> -->
+    <!-- </joint> -->
     <!-- Frame coincident with all-zeros TCP on UR controller -->
     <link name="${prefix}tool0"/>

File: ur5_description/urdf/ur5_robot.urdf.xacro (robot description, xacro)
@@ -9,8 +9,9 @@
   <xacro:ur5_robot prefix="" joint_limited="false"/>
   <link name="world" />
-  <joint name="world_joint" type="fixed">
+  <joint name="world_joint" type="revolute">
     <parent link="world" />
     <child link = "base_link" />
     <origin xyz="0.0 0.0 0.0" rpy="0.0 0.0 0.0" />
+    <axis xyz="0 0 1"/>
   </joint>
 </robot>
